File: hardware/kicad/Orbita26.kicad_sch (KiCad schematic)
At the start: 42 parts, among them J1 Conn_1x4, J2 Conn_01x02, J3 Conn_01x02, J4 Conn_01x04, J5 Conn_01x03, J6 Conn_01x05, J7 Conn_01x04, J8 Conn_01x05, J9 Conn_01x04, Q1 IRLZ44N, U1 TCRT5000, U2 MCP6002-xP, U5 LM393

Commit message: Fixed schem problems & improved readme
Parts:
- C10, C4, C6: footprint (none) -> Capacitor_THT:CP_Radial_D5.0mm_P2.00mm
- C11, C2, C3, C5, C7, C8, C9: footprint (none) -> Capacitor_THT:C_Disc_D5.0mm_W2.5mm_P5.00mm
- J2: footprint (none) -> Connector_AMASS:AMASS_XT30U-M_1x02_P5.0mm_Vertical
- J3: footprint (none) -> TerminalBlock:TerminalBlock_MaiXu_MX126-5.0-02P_1x02_P5.00mm
- J5: footprint (none) -> Connector_JST:JST_XH_B3B-XH-A_1x03_P2.50mm_Vertical
- J6, J8: footprint (none) -> Connector_JST:JST_XH_B5B-XH-A_1x05_P2.50mm_Vertical
- NT1: footprint (none) -> NetTie:NetTie-2_THT_Pad1.0mm
- R1, R11, R12, R13, R15, R16, R17, R18, R3, R6, R7: footprint (none) -> Resistor_THT:R_Axial_DIN0207_L6.3mm_D2.5mm_P7.62mm_Horizontal
- RV2, RV3: footprint (none) -> Potentiometer_THT:Potentiometer_Bourns_3296W_Vertical
- U2, U5: footprint (none) -> Package_DIP:DIP-8_W7.62mm_Socket
Connections:
- net GNDPWR: no longer J3.2 (Pin_2)
- net LED_A: now also R1.2, U1.1 (A)
- net NTC2: now also C7.1, R18.2, TH2.1, U5.3 (+)
- net SENSE: now also C11.1, RV3.1, U1.4 (E)
- net HEATER_LO: now reaches Q1.2 (D), R10.2, R8.2, R9.2
- net HEATER_LO: now also J3.2 (Pin_2)
Other:
- note added: "All the math is in docs/SnailPulse_Math.md on the repo"
- note added: "G = 1 + R17/R16 = 1 + 100k/1k = 101 (40 dB) LPF: f = 1/(2π·100kΩ·470nF) = 3.4 Hz (203 bpm) Pass band 0.16-3.4 Hz ≈ 10-200 bpm"
- note added: "I_LED = (5 − 1.25 V)/220 Ω ≈ 17 mA (max 60 mA)"
- note added: "I²C4: SHT21 0x40 · BMP280 0x76 · MAX30100 0x57 Load: +5V ≈18 mA · +3V3 <25 mA · 14.8V ≤0.34 A (limits 3 A / 3 A / 6 A)"
- note added: "R_heater = 150 Ω/3 = 50 Ω I = 14.8/50 = 0.30 A, P = V²/R = 4.4 W (16.8 V: 5.6 W · 12.8 V: 3.3 W · 1.5 W per 5 W resistor)"
- note added: "V_E = I_photo R_RV3 → tune to ≈1 V DC"
